File: kicad/_autosave-AdderPad.sch (KiCad schematic (older format))
At the start: 18 parts, among them SW1 SW_Push, U1 ProMicro

Commit message: Finished PCB
Parts:
- SW1: footprint Button_Switch_THT:SW_PUSH_6mm -> Keebio-Parts:SW_Tactile_SPST_Angled_MJTP1117
Changed lines of the file:
@@
 F 0 "SW1" H 5200 4235 50  0000 C CNN
 F 1 "SW_Push" H 5200 4144 50  0000 C CNN
-F 2 "Button_Switch_THT:SW_PUSH_6mm" H 5200 4150 50  0001 C CNN
+F 2 "Keebio-Parts:SW_Tactile_SPST_Angled_MJTP1117" H 5200 4150 50  0001 C CNN
 F 3 "~" H 5200 4150 50  0001 C CNN
 	1    5200 3950
