File: kicad/pcb/TurtlePad.kicad_sch (KiCad schematic)
At the start: 23 parts, among them SW1 SW_Push, U1 ProMicro

Commit message: plates and prod files
Connections:
- no-connect marks 4 -> 11
Changed lines of the file:
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@@
   (junction (at 191.77 119.38) (diameter 0) (color 0 0 0 0)
   )
+  (no_connect (at 120.65 135.89))
+  (no_connect (at 120.65 133.35))
+  (no_connect (at 120.65 146.05))
+  (no_connect (at 120.65 143.51))
+  (no_connect (at 120.65 140.97))
+  (no_connect (at 120.65 138.43))
   (no_connect (at 120.65 123.19))
   (no_connect (at 120.65 148.59))
+  (no_connect (at 120.65 151.13))
   (no_connect (at 229.87 111.76))
   (no_connect (at 85.09 125.73))
