File: PCB/rev1.0/TutelPad.kicad_sch (KiCad schematic)
At the start: 15 parts

Commit message: fixing the readme
Parts:
- MX1, MX2, MX3, MX4, MX5, MX6, MX7, MX8: value (none) -> MX; footprint (none) -> 0xcb:SW_Cherry_MX_PCB_1.00u
- OL1: value (none) -> SSD1306
- RGB1, RGB2, RGB3, RGB4: value (none) -> WS2812B
- SW1: value (none) -> SW_Push; footprint (none) -> 0xcb:SW_Tactile_SPST_Angled
- U1: value (none) -> generic-promicro
Other:
- company: (none) -> 0xCB
- title: (none) -> TutelPad
Changed lines of the file:
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@@
 (kicad_sch (version 20211123) (generator eeschema)
   (paper "A4")
+  (title_block
+    (title "TutelPad")
+    (date "2022-04-15")
+    (rev "rev1.0")
+    (company "0xCB")
+  )
   (junction (at 85.09 130.81) (diameter 0) (color 0 0 0 0)
   )
@@
       (effects (font (size 1.524 1.524)))
     )
-    (property "Value" "" (id 1) (at 102.87 118.5926 0)
+    (property "Value" "generic-promicro" (id 1) (at 102.87 118.5926 0)
       (effects (font (size 1.524 1.524)))
     )
@@
       (effects (font (size 1.524 1.524)))
     )
-    (property "Value" "" (id 1) (at 137.9982 43.2054 0)
-      (effects (font (size 0.508 0.508)))
-    )
-    (property "Footprint" "" (id 2) (at 121.285 47.625 0)
+    (property "Value" "MX" (id 1) (at 137.9982 43.2054 0)
+      (effects (font (size 0.508 0.508)))
+    )
+    (property "Footprint" "0xcb:SW_Cherry_MX_PCB_1.00u" (id 2) (at 121.285 47.625 0)
       (effects (font (size 1.524 1.524)) hide)
     )
@@
       (effects (font (size 1.524 1.524)))
     )
-    (property "Value" "" (id 1) (at 155.7782 43.2054 0)
-      (effects (font (size 0.508 0.508)))
-    )
-    (property "Footprint" "" (id 2) (at 139.065 47.625 0)
+    (property "Value" "MX" (id 1) (at 155.7782 43.2054 0)
+      (effects (font (size 0.508 0.508)))
+    )
+    (property "Footprint" "0xcb:SW_Cherry_MX_PCB_1.00u" (id 2) (at 139.065 47.625 0)
       (effects (font (size 1.524 1.524)) hide)
     )
@@
       (effects (font (size 1.524 1.524)))
     )
-    (property "Value" "" (id 1) (at 206.5782 43.2054 0)
-      (effects (font (size 0.508 0.508)))
-    )
-    (property "Footprint" "" (id 2) (at 189.865 47.625 0)
+    (property "Value" "MX" (id 1) (at 206.5782 43.2054 0)
+      (effects (font (size 0.508 0.508)))
+    )
+    (property "Footprint" "0xcb:SW_Cherry_MX_PCB_1.00u" (id 2) (at 189.865 47.625 0)
       (effects (font (size 1.524 1.524)) hide)
     )
@@
       (effects (font (size 1.524 1.524)))
     )
-    (property "Value" "" (id 1) (at 224.3582 43.2054 0)
-      (effects (font (size 0.508 0.508)))
-    )
-    (property "Footprint" "" (id 2) (at 207.645 47.625 0)
+    (property "Value" "MX" (id 1) (at 224.3582 43.2054 0)
+      (effects (font (size 0.508 0.508)))
+    )
+    (property "Footprint" "0xcb:SW_Cherry_MX_PCB_1.00u" (id 2) (at 207.645 47.625 0)
       (effects (font (size 1.524 1.524)) hide)
     )
@@
       (effects (font (size 1.524 1.524)))
     )
-    (property "Value" "" (id 1) (at 137.9982 60.9854 0)
-      (effects (font (size 0.508 0.508)))
-    )
-    (property "Footprint" "" (id 2) (at 121.285 65.405 0)
+    (property "Value" "MX" (id 1) (at 137.9982 60.9854 0)
+      (effects (font (size 0.508 0.508)))
+    )
+    (property "Footprint" "0xcb:SW_Cherry_MX_PCB_1.00u" (id 2) (at 121.285 65.405 0)
       (effects (font (size 1.524 1.524)) hide)
     )
@@
       (effects (font (size 1.524 1.524)))
     )
-    (property "Value" "" (id 1) (at 155.7782 60.9854 0)
-      (effects (font (size 0.508 0.508)))
-    )
-    (property "Footprint" "" (id 2) (at 139.065 65.405 0)
+    (property "Value" "MX" (id 1) (at 155.7782 60.9854 0)
+      (effects (font (size 0.508 0.508)))
+    )
+    (property "Footprint" "0xcb:SW_Cherry_MX_PCB_1.00u" (id 2) (at 139.065 65.405 0)
       (effects (font (size 1.524 1.524)) hide)
     )
@@
       (effects (font (size 1.524 1.524)))
     )
-    (property "Value" "" (id 1) (at 206.5782 60.9854 0)
-      (effects (font (size 0.508 0.508)))
-    )
-    (property "Footprint" "" (id 2) (at 189.865 65.405 0)
+    (property "Value" "MX" (id 1) (at 206.5782 60.9854 0)
+      (effects (font (size 0.508 0.508)))
+    )
+    (property "Footprint" "0xcb:SW_Cherry_MX_PCB_1.00u" (id 2) (at 189.865 65.405 0)
       (effects (font (size 1.524 1.524)) hide)
     )
@@
       (effects (font (size 1.524 1.524)))
     )
-    (property "Value" "" (id 1) (at 224.3582 60.9854 0)
-      (effects (font (size 0.508 0.508)))
-    )
-    (property "Footprint" "" (id 2) (at 207.645 65.405 0)
+    (property "Value" "MX" (id 1) (at 224.3582 60.9854 0)
+      (effects (font (size 0.508 0.508)))
+    )
+    (property "Footprint" "0xcb:SW_Cherry_MX_PCB_1.00u" (id 2) (at 207.645 65.405 0)
       (effects (font (size 1.524 1.524)) hide)
     )
@@
       (effects (font (size 1.27 1.27)) (justify left))
     )
-    (property "Value" "" (id 1) (at 172.72 121.92 0)
+    (property "Value" "WS2812B" (id 1) (at 172.72 121.92 0)
       (effects (font (size 1.27 1.27)) (justify left))
     )
@@
     (in_bom yes) (on_board yes)
     (property "Reference" "SW1" (id 0) (at 105.41 85.471 0))
-    (property "Value" "" (id 1) (at 105.41 87.7824 0))
-    (property "Footprint" "" (id 2) (at 105.41 87.63 0)
+    (property "Value" "SW_Push" (id 1) (at 105.41 87.7824 0))
+    (property "Footprint" "0xcb:SW_Tactile_SPST_Angled" (id 2) (at 105.41 87.63 0)
       (effects (font (size 1.27 1.27)) hide)
     )
@@
       (effects (font (size 1.27 1.27)) (justify left))
     )
-    (property "Value" "" (id 1) (at 187.96 121.92 0)
+    (property "Value" "WS2812B" (id 1) (at 187.96 121.92 0)
       (effects (font (size 1.27 1.27)) (justify left))
     )
@@
       (effects (font (size 1.27 1.27)) (justify left))
     )
-    (property "Value" "" (id 1) (at 203.2 121.92 0)
+    (property "Value" "WS2812B" (id 1) (at 203.2 121.92 0)
       (effects (font (size 1.27 1.27)) (justify left))
     )
@@
       (effects (font (size 1.27 1.27)) (justify left))
     )
-    (property "Value" "" (id 1) (at 218.44 121.92 0)
+    (property "Value" "WS2812B" (id 1) (at 218.44 121.92 0)
       (effects (font (size 1.27 1.27)) (justify left))
     )
@@
     (in_bom yes) (on_board yes) (fields_autoplaced)
     (property "Reference" "OL1" (id 0) (at 173.99 48.4972 90))
-    (property "Value" "" (id 1) (at 173.99 51.0341 90))
+    (property "Value" "SSD1306" (id 1) (at 173.99 51.0341 90))
     (property "Footprint" "0xcb:128x64OLED" (id 2) (at 173.99 52.07 0)
       (effects (font (size 1.27 1.27)) hide)
